File: hardware/can.kicad_sch (KiCad schematic)
At the start: 7 parts

Commit message: worked on it
Parts:
- added J3: DB9_Male_MountingHoles, Connector_Dsub:DSUB-9_Male_Horizontal_P2.77x2.84mm_EdgePinOffset9.90mm_Housed_MountingHolesOffset11.32mm, symbol Connector:DB9_Male_MountingHoles
- added U4: PESD2CANFD24L, Package_TO_SOT_SMD:SOT-23-3, symbol sam-fd:PESD2CANFD24L
- C16, C18, C19: renamed from C?; footprint (none) -> Capacitor_SMD:C_0603_1608Metric; Mfr. (none) -> Murata Electronics; Mfr. No (none) -> GRM188Z71A106KA73D; Mouser No (none) -> 81-GRM188Z71A106KA3D
- C17, C20, C21: renamed from C?; footprint (none) -> Capacitor_SMD:C_0402_1005Metric; Mfr. (none) -> Murata Electronics; Mfr. No (none) -> GRM155R71A104KA01D; Mouser No (none) -> 81-GRM155R71A104KA1D
- U3: renamed from U?; Mfr. (none) -> NXP Semiconductors; Mfr. No (none) -> TJA1443AT/0Z; Mouser No (none) -> 771-TJA1443AT/0Z
Connections:
- net GND: now also J3.3, U4.3
- net CAN_LOW: now reaches U3.12 (CANL)
- net CAN_LOW: now also J3.2, U4.1
- net CAN_HIGH: now reaches U3.13 (CANH)
- net CAN_HIGH: now also J3.7, U4.2
- no-connect marks 0 -> 9
Other:
- moved on the sheet: C16, C17, C18, C19, C20, C21, U3

Commit message: ordered, pray this works
Connections:
- net GND: now also J3.0 (PAD)
- no-connect marks 9 -> 8
Other:
- company: (none) -> Leon Rinkel
- title: (none) -> sam-fd
Changed lines of the file:
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@@
 (kicad_sch (version 20211123) (generator eeschema)
   (paper "A4")
+  (title_block
+    (title "sam-fd")
+    (date "2023-01-27")
+    (rev "2")
+    (company "Leon Rinkel")
+    (comment 1 "leon@rinkel.me")
+    (comment 2 "https://git.leon.fyi/leonrinkel/sam-fd")
+  )
   (junction (at 133.35 83.82) (diameter 0) (color 0 0 0 0)
   )
@@
   (no_connect (at 191.77 105.41))
   (no_connect (at 191.77 97.79))
-  (no_connect (at 199.39 123.19))
   (no_connect (at 191.77 100.33))
   (no_connect (at 191.77 118.11))
@@
     (stroke (width 0) (type default) (color 0 0 0 0))
   )
+  (wire (pts (xy 199.39 123.19) (xy 199.39 130.81))
+    (stroke (width 0) (type default) (color 0 0 0 0))
+  )
   (wire (pts (xy 184.15 113.03) (xy 191.77 113.03))
     (stroke (width 0) (type default) (color 0 0 0 0))
@@
     (effects (font (size 1.27 1.27)) (justify right))
   )
+  (symbol (lib_id "power:GND") (at 199.39 130.81 0) (unit 1)
+    (in_bom yes) (on_board yes)
+    (property "Reference" "#PWR0152" (id 0) (at 199.39 137.16 0)
+      (effects (font (size 1.27 1.27)) hide)
+    )
+    (property "Value" "GND" (id 1) (at 199.39 134.62 0))
+    (property "Footprint" "" (id 2) (at 199.39 130.81 0)
+      (effects (font (size 1.27 1.27)) hide)
+    )
+    (property "Datasheet" "" (id 3) (at 199.39 130.81 0)
+      (effects (font (size 1.27 1.27)) hide)
+    )
+    (pin "1")
+  )
   (symbol (lib_id "power:GND") (at 146.05 96.52 0) (unit 1)
