File: hardware/usb.kicad_sch (KiCad schematic)
At the start: 15 parts

Commit message: worked on it
Parts:
- C12, C14: renamed from C?; footprint (none) -> Capacitor_SMD:C_0402_1005Metric; Mfr. (none) -> Murata Electronics; Mfr. No (none) -> GRM155R61A475MEAAD; Mouser No (none) -> 81-GRM155R61A475MEAD
- C13, C15: renamed from C?; footprint (none) -> Capacitor_SMD:C_0402_1005Metric; Mfr. (none) -> Murata Electronics; Mfr. No (none) -> GRM155R71A104KA01D; Mouser No (none) -> 81-GRM155R71A104KA1D
- D4: renamed from D?; Mfr. (none) -> Littelfuse; Mfr. No (none) -> SP0503BAHTG; Mouser No (none) -> 576-SP0503BAHTG
- D5: renamed from D?; footprint (none) -> Diode_SMD:D_SOD-123; Mfr. (none) -> onsemi; Mfr. No (none) -> MBR130T1G; Mouser No (none) -> 863-MBR130T1G
- D6, D7: renamed from D?; footprint (none) -> LED_SMD:LED_0603_1608Metric; Mfr. (none) -> Lite-On; Mfr. No (none) -> LTST-C190KSKT; Mouser No (none) -> 859-LTST-C190KSKT
- J2: renamed from J?; footprint (none) -> Connector_USB:USB_Micro-B_Molex_47346-0001; Mfr. (none) -> Molex; Mfr. No (none) -> 47346-0001; Mouser No (none) -> 538-47346-0001
- R10: renamed from R?; footprint (none) -> Resistor_SMD:R_0402_1005Metric; Mfr. (none) -> Vishay / Dale; Mfr. No (none) -> CRCW040247K5FKEDC; Mouser No (none) -> 71-CRCW040247K5FKEDC
- R11: renamed from R?; footprint (none) -> Resistor_SMD:R_0402_1005Metric; Mfr. (none) -> Vishay / Dale; Mfr. No (none) -> CRCW04021K00JNEDC; Mouser No (none) -> 71-CRCW04021K00JNEDC
- R12, R13: renamed from R?; footprint (none) -> Resistor_SMD:R_0402_1005Metric; Mfr. (none) -> YAGEO; Mfr. No (none) -> RC0402FR-0768RL; Mouser No (none) -> 603-RC0402FR-0768RL
- R9: renamed from R?; footprint (none) -> Resistor_SMD:R_0402_1005Metric; Mfr. (none) -> Vishay / Dale; Mfr. No (none) -> CRCW040222K1FKEDC; Mouser No (none) -> 71-CRCW040222K1FKEDC
- U2: renamed from U?; Mfr. (none) -> Silicon Labs; Mfr. No (none) -> CP2102N-A02-GQFN28; Mouser No (none) -> 634-CP2102NA02GQFN28
Other:
- moved on the sheet: D4, D5, J2

Commit message: did a little routing
Connections:
- net SHIELD: now reaches J2.6 (Shield)
- no-connect marks 18 -> 17
Changed lines of the file:
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@@
   (no_connect (at 185.42 120.65))
   (no_connect (at 185.42 80.01))
-  (no_connect (at 54.61 104.14))
   (no_connect (at 185.42 115.57))
   (no_connect (at 185.42 123.19))
@@
   )
   (wire (pts (xy 196.85 107.95) (xy 194.31 107.95))
+    (stroke (width 0) (type default) (color 0 0 0 0))
+  )
+  (wire (pts (xy 54.61 104.14) (xy 54.61 106.68))
     (stroke (width 0) (type default) (color 0 0 0 0))
   )
@@
     (stroke (width 0) (type default) (color 0 0 0 0))
   )
+  (label "SHIELD" (at 54.61 106.68 270)
+    (effects (font (size 1.27 1.27)) (justify right bottom))
+  )
   (label "D+" (at 74.93 93.98 0)

Commit message: ordered, pray this works
Parts:
- J2: footprint Connector_USB:USB_Micro-B_Molex_47346-0001 -> sam-fd:USB_Micro-B_Molex_47346-0001
Other:
- company: (none) -> Leon Rinkel
- title: (none) -> sam-fd
Changed lines of the file:
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@@
 (kicad_sch (version 20211123) (generator eeschema)
   (paper "A4")
+  (title_block
+    (title "sam-fd")
+    (date "2023-01-27")
+    (rev "2")
+    (company "Leon Rinkel")
+    (comment 1 "leon@rinkel.me")
+    (comment 2 "https://git.leon.fyi/leonrinkel/sam-fd")
+  )
   (junction (at 72.39 93.98) (diameter 0) (color 0 0 0 0)
   )
@@
     (property "Reference" "J2" (id 0) (at 57.15 81.28 0))
     (property "Value" "USB_B_Micro" (id 1) (at 57.15 83.82 0))
-    (property "Footprint" "Connector_USB:USB_Micro-B_Molex_47346-0001" (id 2) (at 60.96 95.25 0)
-      (effects (font (size 1.27 1.27)) hide)
-    )
+    (property "Footprint" "sam-fd:USB_Micro-B_Molex_47346-0001" (id 2) (at 60.96 95.25 0)
+      (effects (font (size 1.27 1.27)) hide)
+    )
